Commit message: Replace QArm assets: primitive collisions, loadable URDF, real inertias, finger limits
- Collision geometry is now only boxes/cylinders/spheres (43) fitted to the official
  full-resolution meshes; every official vertex lies inside them, so collision is never
  smaller than the visual mesh. Previously Genesis reduced each link to one convex hull,
  which filled the palm between the fingers.
- Named materials: the URDF from 2b8ab95 did not load in Genesis 1.4.4
  ("Missing required attribute name ... Material"), so gripper_demo.py crashed.
- Visual meshes decimated to <= 50k faces: no legacy-parser fallback, 5.4 s load
  instead of 36 s. The 10 full-resolution STLs (byte-identical to Quanser's official
  files) are no longer referenced and are removed.
- Finger joint limits stop at first contact of the two fingers (proximal +-0.1616 rad,
  distal -0.1257 rad). The 2b8ab95 frames were already mirrored correctly; the closing
  scalar (-0.45, ...) overshoots, so the fingers passed through each other.
- Arm inertias from Quanser's QArm Dynamic Parameters, manual joint limits, effort and
  velocity limits, tcp link; small finger masses with the COM at each part's centre.
- Kept the 2b8ab95 gripper frames, all link/joint names and the file path:
  gripper_demo.py runs unchanged.

Generated from the official Quanser BSD-3 files by Jasonartieth/course_project
scripts/model/build_qarm_v2.py @ 7f0bcb5 (see assets/qarm-community/README.md).

Co-Authored-By: Claude Opus 5.5 <noreply@anthropic.com>

File: assets/qarm-community/qarm_with_gripper.urdf (robot description, URDF)
Before this commit: robot QARM, 11 links, 10 joints
Links:
- added link tcp, mass 0.0001
- link BICEP: mass 0.706073338310231 -> 0.4591; geometry collision box size=0.0263703426 0.0300015636 0.0400529665; collision box size=0.047700449 0.071488355 0.100344
- link END-EFFECTOR: mass 0.025331269641348 -> 0.257; geometry collision cylinder length=0.0148 radius=0.0177000006; visual mesh filename=meshes/visual/END-EFFECTOR.stl
- link FOREARM: mass 0.4296669212638 -> 0.269; geometry collision box size=0.00687771131 0.0316998412 0.0333192672; collision box size=0.010960953 0.0161626302 0.0761754855
- link Link1A: mass 0.075987 -> 0.005; geometry collision box size=0.00641137712 0.0155556915 0.0310005087; collision box size=0.0142140308 0.0168800866 0.0343731984
- link Link1B: mass None -> 0.005; geometry collision box size=0.0172103492 0.0185370963 0.0188607208; collision box size=0.0203955923 0.0220499995 0.0422703862
- link Link2A: mass 0.0291073155718739 -> 0.003; geometry collision box size=0.0216999992 0.0230305785 0.0591877194; visual mesh filename=meshes/visual/LINK2A.stl
- link Link2B: mass 0.0291073142953973 -> 0.003; geometry collision box size=0.0216999992 0.0230305785 0.0591877194; visual mesh filename=meshes/visual/LINK2B.stl
- link YAW: mass 0.701518504018672 -> 0.7906; geometry collision box size=0.0117464519 0.0513619396 0.0513619415; collision box size=0.0486889339 0.0604000321 0.0677429802
- link base_link: geometry collision box size=0.0115038517 0.0495427816 0.29664173; collision box size=0.0115046428 0.0233300929 0.327149817
- link gripper_base_link: mass 0.32859 -> 0.005; geometry collision box size=0.00953067896 0.0152161521 0.0342405985; collision box size=0.0118005849 0.0342340368 0.0390023478
Joints:
- added joint tcp_joint: type fixed, parent END-EFFECTOR, child tcp, origin xyz=0 0 0.162 rpy=0 0 0
- joint ELBOW: limit lower=-1.658 upper=1.309 effort=0 velocity=0 -> lower=-1.658063 upper=1.308997 effort=10.6 velocity=1.570796
- joint Joint1A: limit lower=-0.9 upper=0.9 effort=10 velocity=5 -> lower=-0.1616 upper=0.0500 effort=1.9 velocity=2.0; origin xyz=-0.0305 0.0515 0 rpy=0 0 1.5707963267948966 -> xyz=-0.0305 0.0515 0 rpy=0 0 1.57079633
- joint Joint1B: limit lower=-0.9 upper=0.9 effort=10 velocity=5 -> lower=-0.0500 upper=0.1616 effort=1.9 velocity=2.0; origin xyz=0.0305 0.0515 0 rpy=0 0 1.5707963267948966 -> xyz=0.0305 0.0515 0 rpy=0 0 1.57079633
- joint Joint2A: limit lower=-0.9 upper=0.9 effort=10 velocity=5 -> lower=-0.1257 upper=0.0500 effort=1.9 velocity=2.0
- joint Joint2B: limit lower=-0.9 upper=0.9 effort=10 velocity=5 -> lower=-0.1257 upper=0.0500 effort=1.9 velocity=2.0
- joint SHOULDER: limit lower=-1.483 upper=1.483 effort=0 velocity=0 -> lower=-1.483530 upper=1.483530 effort=21.2 velocity=1.570796
- joint WRIST: limit lower=-3.010 upper=3.010 effort=0 velocity=0 -> lower=-2.792527 upper=2.792527 effort=4.1 velocity=1.570796
- joint YAW: limit lower=-2.967 upper=2.967 effort=0 velocity=0 -> lower=-2.967060 upper=2.967060 effort=10.6 velocity=1.570796
- joint gripper_mount: origin xyz=0 0 0 rpy=1.5708 0 1.5708 -> xyz=0 0 0 rpy=1.57079633 0 1.57079633

Commit message: QArm URDF: replace mesh collisions with enclosing boxes/cylinders/spheres
Only the <collision> blocks of assets/qarm-community/qarm_with_gripper.urdf change.
No mesh file is added, removed or modified; visuals, inertials, joints and materials
are byte-identical (checked by stripping the <collision> blocks from both versions).

- Each link's collision mesh is replaced by primitives written directly in the URDF
  (43 in total: boxes, cylinders, spheres), fitted to the full-resolution STL that the
  block referenced, placed with the same <origin>.
- Every STL vertex lies inside the primitives, so collision is never smaller than the
  visual (collision and visual use the same mesh and origin on all 10 links). Checked
  again after writing, by rebuilding the primitives from the written <origin>/<geometry>.
- Genesis no longer reduces each link to one convex hull (the palm between the fingers
  is no longer filled), and since no collision references a >200k-face mesh any more,
  Genesis 1.4.4 no longer falls back to its legacy URDF parser (7.3 s load instead of 36 s).

Generated by Jasonartieth/course_project scripts/model/replace_collisions_with_primitives.py.

Co-Authored-By: Claude Opus 5.5 <noreply@anthropic.com>

File: assets/qarm-community/qarm_with_gripper.urdf (robot description, URDF)
Before this commit: robot QARM, 11 links, 10 joints
Links:
- link BICEP: geometry collision box size=0.02637034 0.03000156 0.04005297; collision box size=0.04770045 0.07148836 0.100344
- link END-EFFECTOR: geometry collision cylinder length=0.0148 radius=0.0177; visual mesh filename=meshes/END-EFFECTOR.STL
- link FOREARM: geometry collision box size=0.006877711 0.03169984 0.03331927; collision box size=0.01096095 0.01616263 0.07617549
- link Link1A: geometry collision box size=0.006411377 0.01555569 0.03100051; collision box size=0.01421403 0.01688009 0.0343732
- link Link1B: geometry collision box size=0.01721035 0.0185371 0.01886072; collision box size=0.02039559 0.02205 0.04227039
- link Link2A: geometry collision box size=0.0217 0.02303058 0.05918772; visual mesh filename=meshes/LINK2A.STL
- link Link2B: geometry collision box size=0.0217 0.02303058 0.05918772; visual mesh filename=meshes/LINK2B.STL
- link YAW: geometry collision box size=0.01174645 0.05136194 0.05136194; collision box size=0.04868893 0.06040003 0.06774298
- link base_link: geometry collision box size=0.01150385 0.04954278 0.2966417; collision box size=0.01150464 0.02333009 0.3271498
- link gripper_base_link: geometry collision box size=0.009530679 0.01521615 0.0342406; collision box size=0.01180058 0.03423404 0.03900235

Commit message: QArm URDF collisions: coarse arm, fine gripper, buried primitives removed
Still only the <collision> blocks change (no mesh files touched). 43 -> 32 primitives
(25 boxes, 6 cylinders, 1 sphere):

- Arm links are coarse: base_link 1, YAW 2, BICEP 4, FOREARM 3, END-EFFECTOR 1
  (was 6 / 4 / 6 / 8 / 1). BICEP and FOREARM keep the fewest primitives that do not
  create false self-contacts: fewer BICEP primitives touched the base in 22 % of random
  poses, fewer FOREARM primitives touched the finger roots when the wrist rotates.
- Gripper is finer: gripper_base_link 10, Link1A 4, Link1B 5, Link2A 1, Link2B 1
  (was 8 / 4 / 4 / 1 / 1).
- Buried primitives removed. Bodies follow Genesis (fixed joints merge links; parent-child
  pairs do not collide). A primitive is dropped when every point of its surface is inside
  another primitive of its body or inside an adjacent body over the whole joint range
  (2 deg steps). Removed: one BICEP box (covered by its neighbour over the full shoulder
  range) and a 0.5 cm3 Link1A box (after growing one Link1A box by 1 mm).
- Collision still encloses every visual vertex (own primitives, or the adjacent body's
  over the whole joint range), re-checked on the written file.

Generated by Jasonartieth/course_project scripts/model/replace_collisions_with_primitives.py
(profile coarse-arm).

Co-Authored-By: Claude Opus 5.5 <noreply@anthropic.com>

File: assets/qarm-community/qarm_with_gripper.urdf (robot description, URDF)
Before this commit: robot QARM, 11 links, 10 joints
Links:
- link BICEP: geometry collision box size=0.07148836 0.07938018 0.1010919; collision cylinder length=0.02758156 radius=0.03723188
- link FOREARM: geometry collision box size=0.02469205 0.04413417 0.09927912; collision box size=0.06530222 0.06939311 0.07617549
- link Link1A: geometry collision box size=0.005409164 0.01985234 0.05049457; collision box size=0.01909041 0.02061038 0.0363732
- link Link1B: geometry collision box size=0.0051625 0.005741029 0.01643748; collision box size=0.01476701 0.01726665 0.01854675
- link YAW: geometry collision box size=0.04868893 0.0677309 0.152806; collision cylinder length=0.02026642 radius=0.07145107
- link base_link: geometry collision box size=0.09586612 0.295675 0.335675; visual mesh filename=meshes/base_link.STL
- link gripper_base_link: geometry collision box size=0.009530679 0.01521615 0.0342406; collision box size=0.01180058 0.03423404 0.03900235
